File: e-ink/EAGLE/e-ink-display-v020/e-ink-display-v020.sch (EAGLE design)
At the start: 170 parts, among them J01M USBUSB-MICROB-PAD-EXTEND, J01S MICROSD, J02S EINKED060SC4, Q01B IRLML6402PbF, Q02B IRLML6402PbF, Q02M MMDT3904, Q2 IRLML6402PbF (DNP), SW01M SWITCHSIDE-SLIDE, U01B BQ24075, U01M STM32F10XRXT6, U01S ADXL345, U02B R8008-33, U03B LT1945-IMS#PBF, U04B LM79L15, U05B LM78L15, U06B LM358-DGKR, U1 MCP73831, Y01M 32kHz, Y02M 8MHz

Commit message: Polishing e-ink-display-v020 to fit my personal taste
Parts:
- removed C02S: 10uF, 6.3V, X5R, kennethlimcp:02-CAP0603-CAP
- removed C03S, C04S: 0.1uF, 6.3V, X5R, kennethlimcp:02-CAP0603-CAP
- removed D01M: BLUE, SparkFun-LED:LED0603
- removed D02M: RGB-LED-CLMVB-FKARGB, Spark:RGB-LED-CLMVB-FKARGB
- removed J01M: USBUSB-MICROB-PAD-EXTEND, Spark:USBUSB-MICROB-PAD-EXTEND
- removed JP1: (no value), SparkFun-Connectors:M08
- removed LOGO1: OSHW-LOGOPAD, kennethlimcp:OSHW-LOGOPAD
- removed R01M, R02M, R03M, R05M: 1K, 1%, kennethlimcp:RESISTOR0603-RES
- removed R02S: 0 Ohm, kennethlimcp:RESISTOR0603-RES
- removed R03S, R04S: 4.7K, 1%, kennethlimcp:RESISTOR0603-RES
- removed TP17M, TP18M: TP1, Spark:TP1
- removed U01S: ADXL345, SparkFun-Sensors:ADXL345
- added J1: (no value), tag-connect:TC2030_SWD-MCP-NL
- added J2: 105017-0001, 105017-0001:105017-0001
- added R112: 10K, rcl:R-EU_R0603
Connections:
- net MCU_USBM renamed MCU_USB_N
- net MCU_USBP renamed MCU_USB_P
- removed net !MCU_RST: C11M.1, JP1.1, R04M.1, S02M.1, U01MRESET.NRST
- removed net JNTRST: JP1.4, U01MPORTB_L.PB4
- removed net JTAG_TRST: R02S.1
- removed net JTCK: JP1.7, U01MPORTA_H.PA14
- removed net JTDI: JP1.6, U01MPORTA_H.PA15
- removed net JTDO: JP1.5, U01MPORTB_L.PB3
- removed net JTMS: D01M.A, JP1.8, U01MPORTA_H.PA13
- removed net MCU_SCL: R04S.1, TP18M.TP, U01MPORTB_L.PB6, U01S.SCL
- removed net MCU_SDA: R03S.1, TP17M.TP, U01MPORTB_L.PB7, U01S.SDA
- removed net N$: J01M.D+, R06M.2, R08M.1
- removed net N$10: R02S.2, U01S.INT1
- removed net N$100: J01M.D-, R07M.2
- removed net N$14: D02M.4, R01M.2
- removed net N$21: R11B.1, TP01B.TP, U02B.EN@1
- removed net N$38: D01M.C, R05M.1
- removed net R02M: D02M.3, R02M.2
- removed net R03M: D02M.2, R03M.2
- removed net RGB_BLUE: R03M.1, U01MPORTA_H.PA8
- removed net RGB_GREEN: R02M.1, U01MPORTA_H.PA10
- removed net RGB_RED: R01M.1, U01MPORTA_H.PA9
- removed net VBUS: C01B.2, C19B.2, J01B.1, J01M.VBUS, R20B.1, U01B.IN, U1.VIN
- new net !RST: C11M.1, J1.!RESET, R04M.1, R112.2, S02M.1, U01MRESET.NRST
- new net MCU_USB_R_N: J2.D-, R07M.2
- new net MCU_USB__R_P: J2.D+, R06M.2, R08M.1
- new net N$20: U06B.-IN1, U06B.OUT1
- new net SWD_CLK: J1.SWCLK/TCK, U01MPORTA_H.PA14
- new net SWD_IO: J1.SWDIO/TMS, U01MPORTA_H.PA13
- new net SWO: J1.SWO/TDO, U01MPORTB_L.PB3
- net +3V3: now also J1.VCC, R112.1; no longer C02S.1, C03S.1, C04S.1, D02M.1, JP1.3, R03S.2, R04S.2, U01S.CS, U01S.VDD, U01S.VS
- net EINK_RL: no longer R13D.1
- net GND: now also J1.GND, J2.GND, J2.HOLES, J2.PADS, R11B.1, TP01B.TP, U02B.EN@1; no longer C02S.2, C03S.2, C04S.2, J01M.GND, JP1.2, R05M.2, U01S.GND@2, U01S.GND@4, U01S.GND@5, U01S.SDO
- net N$6: now also U06B.+IN1
- net VUSB: now also C01B.2, C19B.2, J01B.1, J2.VDD, R20B.1, U01B.IN, U1.VIN
Other:
- note added: "SWD connector"
- note removed: "- CS pulled high for I2C mode - Pins cannot be left floating - Cap values from Sparkfun design"
- note removed: "Accelerometer"
- note removed: "I2C Address table --------------- 0x1010 011x ADXL"
- note removed: "I2C Pull-up"
- note removed: "JTAG"
- note removed: "micro-USB"
